File: f3_backplane.kicad_pcb (KiCad board)
At the start: 4 copper layers, 95.8 x 74 mm, 50 parts, among them J1 PCIEx4_HOST, J2 Bus_M.2_Socket_M, J3 SATA_Backplane, J4 SATA_Backplane, Q1 MMBT3904, U1 NCP45521, U2 NCP45521, U3 NCP45521, U4 NCP45521

Commit message: no DRC errors
Parts:
- removed C13: 22uF, Capacitor_SMD:C_0805_2012Metric
- removed C14, C21, C22, C42, C6: 100nF, Capacitor_SMD:C_0603_1608Metric
- removed Q1: MMBT3904, Package_TO_SOT_SMD:SOT-23
- removed U2, U4: NCP45521, Load_Switches:NCP45521
- added ?: , , F.Cu at (109.2, 69.9)
- added ?: , , F.Cu at (106.3, 66.9)
- added ?: , , F.Cu at (107.8, 70.4)
- added ?: , , F.Cu at (107.8, 66.2)
- added ?: , , F.Cu at (105.7, 68.4)
- added ?: , , F.Cu at (109.2, 66.9)
- added ?: , , F.Cu at (106.3, 69.9)
- added ?: , , F.Cu at (109.8, 68.3)
- added C43: 100nF, Capacitor_SMD:C_0603_1608Metric, B.Cu at (128.2, 81.8)
- added C44: 100nF, Capacitor_SMD:C_0603_1608Metric, B.Cu at (135.4, 48.2)
- added C45: 100nF, Capacitor_SMD:C_0603_1608Metric, B.Cu at (132.0, 81.8)
- added C46: 100nF, Capacitor_SMD:C_0603_1608Metric, B.Cu at (139.4, 48.2)
- C1, C2: value 47u -> 47uF
- C3: value 22u -> 22uF
- C4, C5: value 100n -> 100nF
- U1, U3: value NCP45521 -> STEF512; footprint Load_Switches:NCP45521 -> Load_Switches:TSOT23-8L
- moved C16 23.2 mm to (123.8, 82.8)
- moved C17 23.2 mm to (125.8, 82.6)
- moved C11 22.9 mm to (135.0, 82.6), turned to 90 degrees
- moved C10 20.4 mm to (137.2, 82.8), turned to 90 degrees
- moved U1 19.4 mm to (130.0, 85.2), turned to -90 degrees
- moved C20 15.8 mm to (127.0, 86.0), turned to 90 degrees
- moved C31 14.9 mm to (142.2, 49.0), turned to 90 degrees
- moved C37 14.2 mm to (132.4, 49.0), turned to 90 degrees
- moved U3 12.9 mm to (137.4, 51.6)
- moved C19 12.2 mm to (128.0, 89.0), turned to 0 degrees
- moved C36 11.1 mm to (130.4, 49.2), turned to 90 degrees
- moved C30 10.9 mm to (144.2, 49.2), turned to 90 degrees
- moved R1 6.64 mm to (129.6, 99.6), turned to 0 degrees
- moved C34 6.52 mm to (140.6, 52.4), turned to 90 degrees
- moved C15 5.25 mm to (133.0, 86.0), turned to 90 degrees
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Connections:
- U1 pad 1: +5V -> +12V
- U1 pad 2: /SATA1/PRESENT# -> Net-(U1-SS_12)
- U1 pad 3: +5V -> Net-(U1-SS_5)
- U1 pad 4: GND -> +5V
- U1 pad 6: unconnected-(U1-SR-Pad6) -> GND
- U1 pad 7: /SATA1/SATA_5V -> /SATA1/PRESENT#
- U3 pad 1: +5V -> +12V
- U3 pad 2: /SATA2/PRESENT# -> Net-(U3-SS_12)
- U3 pad 3: +5V -> Net-(U3-SS_5)
- U3 pad 4: GND -> +5V
- U3 pad 6: unconnected-(U3-SR-Pad6) -> GND
- U3 pad 7: /SATA2/SATA_5V -> /SATA2/PRESENT#
Routing:
- net +5V: track 66.5 -> 19.0 mm, vias 35 -> 34
- net /SATA2/PRESENT#: track 60.7 -> 31.4 mm, vias 2 -> 1
- net /Connector/B30: track 19.0 -> 0.00 mm, vias 1 -> 0
- net /Connector/B31: track 15.4 -> 0.00 mm, vias 1 -> 0
- net /SATA1/PRESENT#: track 26.1 -> 15.6 mm, vias 2 -> 1
- net GND: track 128.1 -> 136.4 mm, vias 142 -> 261
- net Net-(U1-SS_5): track 0.00 -> 3.00 mm
- net Net-(U3-SS_5): track 0.00 -> 3.00 mm
- net Net-(U3-SS_12): track 0.00 -> 3.00 mm
- net Net-(U1-SS_12): track 0.00 -> 2.85 mm

Commit message: revision V1.1
Other:
- board text added: "Modified by Endre Vestå"
- board text added: "Original by codedbearder.com"
- board text removed: "codedbearder.com"
